File: X15-ESC-Adapter.sch (EAGLE design)
At the start: 6 parts, among them J1 IPBT-103-H1-T-S, J2 IPBT-103-H1-T-S, J3 IPBT-103-H1-T-S, J4 IPBT-103-H1-T-S

Commit message: Second Version - Schematic V1
Need schematic review
Parts:
- removed U$1: LUMENIER, X15-ESC-Adapter:LUMENIER
- added BACKPLANE_CONNECTIONS: BACKPLANE_ESC_ADAPTER_PWRBKP, X15-ESC-Adapter:BACKPLANE_ESC_ADAPTER_PWRBKP
- added H1, H2, H3, H4: 6-32-HOLE, X15-ESC-Adapter:6-32-HOLE
- renumbered LUMENIER to LUMENIER_ESC
Connections:
- net N$25 renamed GND
- removed net N$26: LUMENIER_ESC.VIN
- new net 12V: BACKPLANE_CONNECTIONS.12V, LUMENIER_ESC.VIN
- new net N$1: BACKPLANE_CONNECTIONS.GND

Commit message: First Final Version of Board
Finished first version of board
Connections:
- removed net N$1: BACKPLANE_CONNECTIONS.GND
- net ESC1_B: now also LUMENIER_ESC.M1P1; no longer LUMENIER_ESC.M1P3
- net ESC1_R: now also LUMENIER_ESC.M1P3; no longer LUMENIER_ESC.M1P1
- net ESC2_B: now also LUMENIER_ESC.M2P1; no longer LUMENIER_ESC.M2P3
- net ESC2_R: now also LUMENIER_ESC.M2P3; no longer LUMENIER_ESC.M2P1
- net ESC3_B: now also J3.1, LUMENIER_ESC.M3P1; no longer J3.3, LUMENIER_ESC.M3P3
- net ESC3_R: now also J3.3, LUMENIER_ESC.M3P3; no longer J3.1, LUMENIER_ESC.M3P1
- net ESC4_B: now also J4.1, LUMENIER_ESC.M4P1; no longer J4.3, LUMENIER_ESC.M4P3
- net ESC4_R: now also J4.3, LUMENIER_ESC.M4P3; no longer J4.1, LUMENIER_ESC.M4P1
- net GND: now also BACKPLANE_CONNECTIONS.GND

Commit message: Parts Replaced with New Versions
Parts:
- BACKPLANE_CONNECTIONS: value BACKPLANE_ESC_ADAPTER_PWRBKP -> IPS1-112-01-L-DBKP; device X15-ESC-Adapter:BACKPLANE_ESC_ADAPTER_PWRBKP -> X15-ESC-Adapter:IPS1-112-01-L-DBKP
Changed lines of the file:
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@@
 <parts>
 <part name="FRAME1" library="SparkFun-Aesthetics" library_urn="urn:adsk.eagle:library:507" deviceset="FRAME-A4L" device=""/>
-<part name="J4" library="X15-ESC-Adapter" deviceset="IPBT-103-H1-T-S" device=""/>
-<part name="J3" library="X15-ESC-Adapter" deviceset="IPBT-103-H1-T-S" device=""/>
-<part name="J2" library="X15-ESC-Adapter" deviceset="IPBT-103-H1-T-S" device=""/>
-<part name="J1" library="X15-ESC-Adapter" deviceset="IPBT-103-H1-T-S" device=""/>
-<part name="LUMENIER_ESC" library="X15-ESC-Adapter" deviceset="LUMENIER" device="" package3d_urn="urn:adsk.eagle:package:24294694/3"/>
-<part name="BACKPLANE_CONNECTIONS" library="X15-ESC-Adapter" deviceset="BACKPLANE_ESC_ADAPTER_PWR" device="BKP"/>
+<part name="J4" library="X15-ESC-Adapter" deviceset="IPBT-103-H1-T-S" device="" package3d_urn="urn:adsk.eagle:package:37886187/2"/>
+<part name="J3" library="X15-ESC-Adapter" deviceset="IPBT-103-H1-T-S" device="" package3d_urn="urn:adsk.eagle:package:37886187/2"/>
+<part name="J2" library="X15-ESC-Adapter" deviceset="IPBT-103-H1-T-S" device="" package3d_urn="urn:adsk.eagle:package:37886187/2"/>
+<part name="J1" library="X15-ESC-Adapter" deviceset="IPBT-103-H1-T-S" device="" package3d_urn="urn:adsk.eagle:package:37886187/2"/>
+<part name="LUMENIER_ESC" library="X15-ESC-Adapter" deviceset="LUMENIER" device="" package3d_urn="urn:adsk.eagle:package:37886188/1"/>
+<part name="BACKPLANE_CONNECTIONS" library="X15-ESC-Adapter" library_urn="urn:adsk.eagle:library:38003364" deviceset="IPS1-112-01-L-D" device="BKP" package3d_urn="urn:adsk.eagle:package:37886186/4"/>
 <part name="SUPPLY1" library="supply2" library_urn="urn:adsk.eagle:library:372" deviceset="GND" device=""/>
-<part name="H1" library="X15-ESC-Adapter" deviceset="6-32-HOLE" device="" package3d_urn="urn:adsk.eagle:package:24384748/2"/>
-<part name="H2" library="X15-ESC-Adapter" deviceset="6-32-HOLE" device="" package3d_urn="urn:adsk.eagle:package:24384748/2"/>
-<part name="H3" library="X15-ESC-Adapter" deviceset="6-32-HOLE" device="" package3d_urn="urn:adsk.eagle:package:24384748/2"/>
-<part name="H4" library="X15-ESC-Adapter" deviceset="6-32-HOLE" device="" package3d_urn="urn:adsk.eagle:package:24384748/2"/>
+<part name="H1" library="X15-ESC-Adapter" deviceset="6-32-HOLE" device="" package3d_urn="urn:adsk.eagle:package:37886189/1"/>
+<part name="H2" library="X15-ESC-Adapter" deviceset="6-32-HOLE" device="" package3d_urn="urn:adsk.eagle:package:37886189/1"/>
+<part name="H3" library="X15-ESC-Adapter" deviceset="6-32-HOLE" device="" package3d_urn="urn:adsk.eagle:package:37886189/1"/>
+<part name="H4" library="X15-ESC-Adapter" deviceset="6-32-HOLE" device="" package3d_urn="urn:adsk.eagle:package:37886189/1"/>
 </parts>
 <sheets>

Commit message: Fixed strange things
Parts:
- BACKPLANE_CONNECTIONS: value IPS1-112-01-L-DBKP -> IPS1-112-01-L-D; device X15-ESC-Adapter:IPS1-112-01-L-DBKP -> X15-ESC-Adapter:IPS1-112-01-L-D
Changed lines of the file:
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@@
 <part name="J1" library="X15-ESC-Adapter" deviceset="IPBT-103-H1-T-S" device="" package3d_urn="urn:adsk.eagle:package:37886187/2"/>
 <part name="LUMENIER_ESC" library="X15-ESC-Adapter" deviceset="LUMENIER" device="" package3d_urn="urn:adsk.eagle:package:37886188/1"/>
-<part name="BACKPLANE_CONNECTIONS" library="X15-ESC-Adapter" library_urn="urn:adsk.eagle:library:38003364" deviceset="IPS1-112-01-L-D" device="BKP" package3d_urn="urn:adsk.eagle:package:37886186/4"/>
 <part name="SUPPLY1" library="supply2" library_urn="urn:adsk.eagle:library:372" deviceset="GND" device=""/>
 <part name="H1" library="X15-ESC-Adapter" deviceset="6-32-HOLE" device="" package3d_urn="urn:adsk.eagle:package:37886189/1"/>
@@
 <part name="H3" library="X15-ESC-Adapter" deviceset="6-32-HOLE" device="" package3d_urn="urn:adsk.eagle:package:37886189/1"/>
 <part name="H4" library="X15-ESC-Adapter" deviceset="6-32-HOLE" device="" package3d_urn="urn:adsk.eagle:package:37886189/1"/>
+<part name="BACKPLANE_CONNECTIONS" library="X15-ESC-Adapter" deviceset="IPS1-112-01-L-D" device="" package3d_urn="urn:adsk.eagle:package:38090775/2"/>
 </parts>
 <sheets>
@@
 <attribute name="NAME" x="152.4" y="111.76" size="1.778" layer="95"/>
 </instance>
-<instance part="BACKPLANE_CONNECTIONS" gate="G$1" x="218.44" y="132.08" smashed="yes">
-<attribute name="NAME" x="215.9" y="129.54" size="1.27" layer="95" rot="R90"/>
-</instance>
 <instance part="SUPPLY1" gate="GND" x="218.44" y="104.14" smashed="yes">
 <attribute name="VALUE" x="216.535" y="100.965" size="1.778" layer="96"/>
@@
 <attribute name="NAME" x="91.44" y="132.08" size="1.016" layer="95" align="bottom-center"/>
 <attribute name="VALUE" x="91.44" y="127" size="1.016" layer="95" align="top-center"/>
+</instance>
+<instance part="BACKPLANE_CONNECTIONS" gate="G$1" x="218.44" y="132.08" smashed="yes">
+<attribute name="NAME" x="215.9" y="129.54" size="1.27" layer="95" rot="R90"/>
 </instance>
 </instances>
@@
 <net name="12V" class="0">
 <segment>
-<pinref part="BACKPLANE_CONNECTIONS" gate="G$1" pin="12V"/>
 <wire x1="218.44" y1="144.78" x2="218.44" y2="154.94" width="0.1524" layer="91"/>
 <label x="218.44" y="154.94" size="1.778" layer="95" xref="yes"/>
+<pinref part="BACKPLANE_CONNECTIONS" gate="G$1" pin="12V"/>
 </segment>
 <segment>
@@
 </segment>
 <segment>
-<pinref part="BACKPLANE_CONNECTIONS" gate="G$1" pin="GND"/>
 <wire x1="218.44" y1="119.38" x2="218.44" y2="106.68" width="0.1524" layer="91"/>
 <pinref part="SUPPLY1" gate="GND" pin="GND"/>
 <label x="218.44" y="106.68" size="1.778" layer="95" rot="R270"/>
-</segment>
-</net>
+<pinref part="BACKPLANE_CONNECTIONS" gate="G$1" pin="GND"/>
+</segment>
+</net>
